File: Dropsense_V2/PCB/SENDER/dropsense_SENDER_v2/dropsense_v2.kicad_sch (KiCad schematic)
At the start: 35 parts, among them J1 USB_B_Micro, J2 Conn_01x02, J3 Micro_SD_Card_Det_Hirose_DM3AT, J4 Conn_01x06_Pin, U1 ESP32-S3-WROOM-1, U2 TP4056-42-ESOP8, U3 ME6211C33M5, U4 MPU-6050

Commit message: started work on dropsense sender and reciever new pcb
Parts:
- removed D3, D4: SS14, Diode_SMD:D_SMA, symbol Diode:SS14
- added C11, C13: 10uF, Capacitor_SMD:C_0805_2012Metric, symbol Device:C
- added C12: 1uF, Capacitor_SMD:C_0805_2012Metric, symbol Device:C
- added R12, R13: 22R, Resistor_SMD:R_0805_2012Metric, symbol Device:R
- R1: value 1.2kR -> 3.3kR
Connections:
- net 3V3: now also C11.1
- net D+: now also R13.2; no longer U1.14 (USB_D+)
- net D-: now also R12.2; no longer U1.13 (USB_D-)
- net EN: now also C12.1
- net GND: now also C1.1, J3.11 (SHIELD), C11.2, C12.2, C13.2; no longer C1.2
- net VBAT: now also C1.2, U3.1 (V_{IN}), U3.3 (CE), C13.1
- net MPU_INTERUPT: now reaches U1.15 (IO3)
- net MPU_INTERUPT: now also U4.12 (INT)
- net at J1.1 (VBUS): now also R2.1, R3.1, U2.4 (V_{CC}), U2.8 (CE)
- removed net VBUS: J1.4 (ID), R2.1, R3.1, U2.4 (V_{CC}), U2.8 (CE)
- removed net V_IN: C1.1, U3.1 (V_{IN}), U3.3 (CE)
- new net: R13.1, U1.14 (USB_D+)
- new net: R12.1, U1.13 (USB_D-)
