File: Dropsense_V2/PCB/RECIEVER/Dropsense_reciever_V2/dropsense_reciever_v2.kicad_sch (KiCad schematic)
At the start: 29 parts, among them J1 USB_B_Micro, J2 Battery_conn, J3 1.8inch TFT connector, U1 TP4056-42-ESOP8, U2 ME6211C33M5, U3 ESP32-S3-WROOM-1

Commit message: made dropsense reciever pcb
Parts:
- C1, C2, C3, C4, C5, C6: footprint (none) -> Capacitor_SMD:C_0805_2012Metric
- D3, D4: footprint (none) -> LED_SMD:LED_0805_2012Metric
- J1: footprint (none) -> Connector_USB:USB_Micro-B_Amphenol_10118194-0001LF_Horizontal
- J2: footprint (none) -> Connector_JST:JST_XH_B2B-XH-A_1x02_P2.50mm_Vertical
- R1, R2, R3, R4, R5: footprint (none) -> Resistor_SMD:R_0805_2012Metric
Connections:
- net GND: now also C5.2, C6.2
- net 3V3 renamed 3v3
- net 3v3: no longer C5.2, C6.2
Other:
- moved on the sheet: R8
